File: Electronics/IMU.kicad_sch (KiCad schematic)
At the start: 9 parts, among them J1 Conn_01x07_Socket, J2 LCD Display, U1 RASPBERRY_PI_ZERO_2_W

Commit message: IMU testing + schematic fix
Connections:
- net IMU_SCL: now also J2.2 (Pin_2), R4.2, U1.5 (GPIO3/SCL); no longer U1.29 (GPIO5)
- net IMU_SDA: now also J2.1 (Pin_1), R3.2, U1.3 (GPIO2/SDA1); no longer U1.31 (GPIO6)
- removed net LCD_SCL: J2.2 (Pin_2), R4.2, U1.26 (GPIO7/SPI_~{CE1})
- removed net LCD_SDA: J2.1 (Pin_1), R3.2, U1.24 (GPIO8/SPI_~{CE0})
- no-connect marks 33 -> 35
Changed lines of the file:
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@@
+	)
+	(junction
+		(at 99.06 78.74)
+		(diameter 0)
+		(color 0 0 0 0)
+	)
+	(junction
+		(at 166.37 58.42)
+		(diameter 0)
+		(color 0 0 0 0)
+	)
+	(junction
+		(at 68.58 83.82)
+		(diameter 0)
+		(color 0 0 0 0)
+	)
+	(junction
+		(at 171.45 63.5)
+		(diameter 0)
+		(color 0 0 0 0)
+	)
+	(junction
+		(at 168.91 114.3)
+		(diameter 0)
+		(color 0 0 0 0)
+	)
+	(junction
+		(at 168.91 111.76)
+		(diameter 0)
+		(color 0 0 0 0)
 	)
 	(junction
@@
 	)
 	(junction
-		(at 166.37 58.42)
-		(diameter 0)
-		(color 0 0 0 0)
-	)
-	(junction
-		(at 171.45 63.5)
-		(diameter 0)
-		(color 0 0 0 0)
-	)
-	(junction
-		(at 168.91 114.3)
-		(diameter 0)
-		(color 0 0 0 0)
-	)
-	(junction
-		(at 168.91 111.76)
-		(diameter 0)
-		(color 0 0 0 0)
-	)
-	(junction
 		(at 200.66 113.03)
 		(diameter 0)
@@
 	)
 	(junction
-		(at 68.58 83.82)
+		(at 91.44 78.74)
+		(diameter 0)
+		(color 0 0 0 0)
+	)
+	(junction
+		(at 101.6 81.28)
 		(diameter 0)
 		(color 0 0 0 0)
@@
 		(color 0 0 0 0)
 	)
-	(junction
-		(at 91.44 78.74)
-		(diameter 0)
-		(color 0 0 0 0)
-	)
-	(no_connect
-		(at 104.14 73.66)
-	)
 	(no_connect
 		(at 104.14 101.6)
@@
 	)
 	(no_connect
-		(at 104.14 71.12)
-	)
-	(no_connect
 		(at 214.63 88.9)
 	)
@@
 	)
 	(no_connect
+		(at 104.14 78.74)
+	)
+	(no_connect
+		(at 104.14 81.28)
+	)
+	(no_connect
 		(at 165.1 96.52)
 	)
@@
 	)
 	(no_connect
+		(at 104.14 86.36)
+	)
+	(no_connect
 		(at 165.1 86.36)
 	)
@@
 	)
 	(no_connect
+		(at 104.14 83.82)
+	)
+	(no_connect
 		(at 165.1 88.9)
 	)
@@
 	(wire
 		(pts
-			(xy 91.44 78.74) (xy 104.14 78.74)
-		)
-		(stroke
-			(width 0)
-			(type default)
-		)
-	)
-	(wire
-		(pts
 			(xy 170.18 114.3) (xy 168.91 114.3)
 		)
@@
 	(wire
 		(pts
+			(xy 99.06 78.74) (xy 99.06 73.66)
+		)
+		(stroke
+			(width 0)
+			(type default)
+		)
+	)
+	(wire
+		(pts
 			(xy 165.1 58.42) (xy 166.37 58.42)
 		)
@@
 	(wire
 		(pts
+			(xy 101.6 71.12) (xy 104.14 71.12)
+		)
+		(stroke
+			(width 0)
+			(type default)
+		)
+	)
+	(wire
+		(pts
 			(xy 82.55 78.74) (xy 91.44 78.74)
 		)
@@
 	(wire
 		(pts
+			(xy 68.58 83.82) (xy 99.06 83.82)
+		)
+		(stroke
+			(width 0)
+			(type default)
+		)
+	)
+	(wire
+		(pts
 			(xy 91.44 64.77) (xy 91.44 68.58)
 		)
@@
 	(wire
 		(pts
-			(xy 91.44 86.36) (xy 104.14 86.36)
+			(xy 91.44 86.36) (xy 101.6 86.36)
 		)
 		(stroke
@@
 	(wire
 		(pts
-			(xy 68.58 81.28) (xy 104.14 81.28)
-		)
-		(stroke
-			(width 0)
-			(type default)
-		)
-	)
-	(wire
-		(pts
-			(xy 68.58 83.82) (xy 104.14 83.82)
-		)
-		(stroke
-			(width 0)
-			(type default)
-		)
-	)
-	(wire
-		(pts
 			(xy 58.42 83.82) (xy 68.58 83.82)
 		)
@@
 	(wire
 		(pts
+			(xy 101.6 81.28) (xy 101.6 86.36)
+		)
+		(stroke
+			(width 0)
+			(type default)
+		)
+	)
+	(wire
+		(pts
+			(xy 91.44 78.74) (xy 99.06 78.74)
+		)
+		(stroke
+			(width 0)
+			(type default)
+		)
+	)
+	(wire
+		(pts
+			(xy 68.58 81.28) (xy 101.6 81.28)
+		)
+		(stroke
+			(width 0)
+			(type default)
+		)
+	)
+	(wire
+		(pts
 			(xy 68.58 95.25) (xy 68.58 99.06)
 		)
@@
 	(wire
 		(pts
+			(xy 101.6 81.28) (xy 101.6 71.12)
+		)
+		(stroke
+			(width 0)
+			(type default)
+		)
+	)
+	(wire
+		(pts
 			(xy 53.34 66.04) (xy 58.42 66.04)
 		)
@@
 	(wire
 		(pts
+			(xy 99.06 73.66) (xy 104.14 73.66)
+		)
+		(stroke
+			(width 0)
+			(type default)
+		)
+	)
+	(wire
+		(pts
 			(xy 168.91 111.76) (xy 165.1 111.76)
 		)
@@
 		)
 		(stroke
+			(width 0)
+			(type default)
+		)
+	)
+	(wire
+		(pts
+			(xy 99.06 83.82) (xy 99.06 78.74)
+		)
+		(stroke
